File: frmw_dcin_big/frmw_dcin_big.kicad_sch (KiCad schematic)
At the start: 53 parts, among them J2 SMART, M1 AltmodeFriend, Q1 SI4909, Q2 2N7002, Q3 2N7002, Q4 2N7002, Q5 SI4909, Q6 2N7002, Q7 SI4909, U1 SY6280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

Commit message: design: reviewed. added a proper circuit for HP/Dell center pin detection, did BOM optimizations, recalculated SY6280 resistors, yote via-in-pad, improved tracks and fills, updated USB-C footprint
Parts:
- added C12, C13, C14, C15: 10nF, Capacitor_SMD:C_0402_1005Metric, symbol Device:C_Small
- added D2: 3V6, Diode_SMD:D_0805_2012Metric, symbol Device:D_Zener_Small
- added R11, R14: 1K8, Resistor_SMD:R_0402_1005Metric, symbol Device:R_Small
- added R2: 20K, Resistor_SMD:R_0402_1005Metric, symbol Device:R_Small
- added R3: 5K1, Resistor_SMD:R_0402_1005Metric, symbol Device:R_Small
- added R5: 0R, Resistor_SMD:R_0402_1005Metric, symbol Device:R_Small
- C4: footprint Capacitor_SMD:C_0603_1608Metric -> Capacitor_SMD:C_0805_2012Metric
- D1: value D_Small -> Schottky 1A
- ISET1: value x -> 5K1; footprint Resistor_SMD:R_0603_1608Metric -> Resistor_SMD:R_0402_1005Metric
- Q2, Q3, Q4, Q6: symbol Device:Q_PMOS_GSD -> Device:Q_NMOS_GSD
- R1: value 0R -> NC
- R19: value 1K -> 20K; footprint Resistor_SMD:R_0603_1608Metric -> Resistor_SMD:R_0402_1005Metric
- R22: value 1K -> 1K8
- R23: value 10K -> 20K
Connections:
- net +3.3V: no longer C3.1, C4.1
- net +5V: now also C3.1, C4.1
- net GND: now also Q2.2 (S), Q3.2 (S), Q4.2 (S), Q6.2 (S), R19.2, C12.2, C13.2, C14.2, C15.2, D2.2 (A), R2.2; no longer Q2.3 (D), Q3.3 (D), Q4.3 (D), Q6.3 (D)
- net HD_PSID: now also D2.1 (K), R2.1, R5.2; no longer M1.3 (BOOT_(27))
- net SY_EN: now also M1.4 (GP0); no longer M1.5 (GP1)
- net VBUS: now also C12.1, C13.1, C14.1, C15.1, R11.1, R14.1; no longer R19.1
- net PSID_PU_EN: now reaches M1.6 (GP2)
- net PSID_PU_EN: now also R3.1
- net at R18.2: now also Q6.3 (D); no longer Q6.2 (S)
- net at R8.2: now also Q3.3 (D); no longer Q3.2 (S)
- net at ISET1.1, U1.3 (ISET): now also R19.1
- net at Q5.2 (G), R12.2: now also Q2.3 (D); no longer Q2.2 (S)
- new net: Q4.3 (D), R11.2, R14.2
- new net PSID_R: M1.3 (BOOT_(27)), R3.2, R5.1
Other:
- note added: "(4.06k Iset resistor)"
- note added: "PSID circuit"
- note added: "R2/D2 for HP ADC limiting D3 for Dell one-wire"
- note added: "TODO [x] add ID circuits [n] add LEDs (+ onto testpoints) [n] add buttons? (new AF will have a neopixel and buttons)"
- note added: "USB-C plug capacitors"
- note removed: "FrmW card doesn't need this for sure"
- note removed: "FrmW card doesn't need this ig? TODO on any details, of course"
- note removed: "Lenovo/generic input"
- note removed: "PC PSU input"
- note removed: "TODO [ ] add ID circuits [ ] add LEDs (+ onto testpoints) [ ] add buttons? new AF will have a LED and buttons tho"
- note removed: "TODO calc R(iset)"
- note removed: "idk about this one"
- moved on the sheet: C1, C2, R22, R23
