File: frmw_dcin_big/frmw_dcin_big.kicad_pcb (KiCad board)
At the start: 2 copper layers, 41.5 x 24 mm, 64 parts, among them J2 SMART, M1 AltmodeFriend, Q1 SI4909, Q2 2N7002, Q3 2N7002, Q4 2N7002, Q5 SI4909, Q6 2N7002, Q7 SI4909, U1 SY6280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

Commit message: Changed to 4 layers
Routing:
- added copper zone on In1.Cu, net GND
- added copper zone on In2.Cu, net GND
Other:
- copper layers 2 -> 4
Changed lines of the file:
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@@
 	(layers
 		(0 "F.Cu" signal)
+		(1 "In1.Cu" signal)
+		(2 "In2.Cu" signal)
 		(31 "B.Cu" signal)
 		(32 "B.Adhes" user "B.Adhesive")
@@
 			)
 			(layer "dielectric 1"
+				(type "prepreg")
+				(thickness 0.1)
+				(material "FR4")
+				(epsilon_r 4.5)
+				(loss_tangent 0.02)
+			)
+			(layer "In1.Cu"
+				(type "copper")
+				(thickness 0.035)
+			)
+			(layer "dielectric 2"
 				(type "core")
-				(thickness 0.71)
+				(thickness 0.44)
+				(material "FR4")
+				(epsilon_r 4.5)
+				(loss_tangent 0.02)
+			)
+			(layer "In2.Cu"
+				(type "copper")
+				(thickness 0.035)
+			)
+			(layer "dielectric 3"
+				(type "prepreg")
+				(thickness 0.1)
 				(material "FR4")
 				(epsilon_r 4.5)
@@
 		(net 2)
 		(net_name "GND")
-		(layers "F&B.Cu")
+		(layers "F.Cu" "In1.Cu" "In2.Cu" "B.Cu")
 		(hatch edge 0.5)
 		(connect_pads yes
